File: kicad/ch32v003j4m6-rx8900ce/ch32v003j4m6-rx8900.kicad_pcb (KiCad board)
At the start: 2 copper layers, 39.2 x 19 mm, 18 parts, among them J1 Conn_01x03, SW1 SW_Push, U1 CH32V003JxMx, U2 RX8900CE

Commit message: Update kicad files
Parts:
- removed D3: D, Diode_SMD:D_SOD-123F
Connections:
- BT1 pad 1: +BATT0 -> +BATT
- C3 pad 2: +BATT1 -> +BATT
- SW1 pad 2: +BATT1 -> +BATT
- U2 pad 3: +BATT1 -> +BATT
Routing:
- net +BATT: track 0.00 -> 54.3 mm, vias 0 -> 6
- net +BATT1: track 49.4 -> 0.00 mm, vias 5 -> 0
- net +BATT0: track 5.94 -> 0.00 mm, vias 1 -> 0
- net GND: track 22.4 -> 23.6 mm, vias 4 -> 19
- net +3.3V: track 89.4 -> 90.3 mm
- added copper zone on F.Cu, net GND
- removed copper zone on F.Cu, net +3.3V

Commit message: Update pcb/sch
Parts:
- removed C4: C, Capacitor_SMD:C_0603_1608Metric
Routing:
- net Net-(U1-PC2): track 22.3 -> 16.0 mm
- net Net-(D2-A): track 16.3 -> 11.3 mm
- net GND: track 23.6 -> 20.0 mm, vias 19 -> 13
- net +3.3V: track 90.3 -> 87.2 mm
- net +BATT: track 54.3 -> 52.7 mm, vias 6 -> 3
- added copper zone on B.Cu, net +BATT
Other:
- board text added: "Gathering CLOCK ver 0.4 @task_jp"
- board text removed: "Gathering CLOCK ver 0.3 @task_jp"
